Commit message: fixed camera joint

File: urdf/a2.urdf (robot description, URDF)
Before this commit: robot a2, 21 links, 20 joints
Links:
- added link front_camera_optical_frame
Joints:
- added joint front_camera_optical_joint: type fixed, parent camera_link, child front_camera_optical_frame, origin xyz=0 0 0 rpy=-1.5708 0 -1.5708
- joint front_camera_joint: origin xyz=0.3421785 0.0336742 0.0513862 rpy=1.5708 0.0 1.5708 -> xyz=0.3421785 0.0336742 0.0513862 rpy=0.0 0.0 0.0
